File: Schematics/Clock_Updated_3_board2.sch (EAGLE design)
At the start: 53 parts, among them U1 ATMEGA328P

Commit message: found out vdd and ledvdd were switched
Parts:
- added R17, R18: 180, SparkFun-Resistors:180OHM1/10W1%(0603)
- added S3: (no value), SparkFun-Electromechanical:TAC_SWITCHPTH
- renumbered C12 to LED12CAP
Connections:
- new net POWER: C16.1, IC1.OUT, U1.AREF, U1.AVCC
- new net RESET_S: S3.3, U1.PD4(XCK/T0)
- net GND: now also S3.1
- net N$37: now also R17.2, R18.2; no longer C16.1, IC1.OUT
- net PIN14: now also U1.PD6(AIN0); no longer U1.PB0(ICP)
- net PIN15: now also U1.PD7(AIN1); no longer U1.PB1(OC1A)
- net PIN16: now also U1.PB0(ICP); no longer U1.PB2(SS/OC1B)
Other:
- moved on the sheet: Y1
