File: Schematics/final/Clock_Updated_3_Nets.brd (EAGLE design)
At the start: 50.8 x 50.8 mm, 51 parts, among them U1 ATMEGA328P, U2 V_REG_317DPACK

Commit message: changed wires
Parts:
- removed C11, C12: 0.1uF, SparkFun-Capacitors:0603-CAP
- removed CN2: (no value), adafruit:DCJACK_2MM_SMT
- removed LED11, LED12: WS2812, adafruit:WS2812
- added C17, C18: 0.1uF, SparkFun-Capacitors:0603-CAP
- added LED13, LED14: WS2812, adafruit:WS2812
- added U$2: CUI_PJ-102A, con-dc-jack:CUI_DCJACK_PCB
- moved R11 143.7 mm to (1.52, -106.7), flipped to the top, turned to 0 degrees
- moved R12 142.5 mm to (4.57, -106.7), flipped to the top, turned to 0 degrees
- moved R10 136.0 mm to (16.8, -103.6), flipped to the top
- moved LED10 135.0 mm to (11.7, -97.5), flipped to the top, turned to 0 degrees
- moved C10 135.0 mm to (10.7, -103.6), flipped to the top
- moved R9 132.5 mm to (13.7, -103.6), flipped to the top, turned to 0 degrees
- moved C9 131.6 mm to (7.62, -103.6), flipped to the top
- moved LED9 129.3 mm to (3.05, -97.5), flipped to the top, turned to 0 degrees
- moved C8 128.4 mm to (4.57, -103.6), flipped to the top
- moved C7 123.4 mm to (1.52, -103.6), flipped to the top, turned to 0 degrees
- moved R8 108.8 mm to (4.57, -81.3), flipped to the top, turned to 0 degrees
- moved LED8 108.4 mm to (11.7, -87.9), flipped to the top, turned to 0 degrees
- moved C3 103.5 mm to (1.52, -78.2), flipped to the top, turned to 0 degrees
- moved LED7 102.7 mm to (3.05, -87.9), flipped to the top, turned to 0 degrees
- moved R7 102.2 mm to (1.52, -81.3), flipped to the top, turned to 0 degrees
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Connections:
- removed net N$22 (its old number): C11.1, LED11.LEDVDD, R11.2
- removed net N$23 (its old number): C12.1, LED12.LEDVDD, R12.2
- removed net N$24 (its old number): LED11.DI, LED12.DO
- new net : U$2.CASE
- new net N$12: LED3.LEDVDD, R5.2
- new net N$15: C5.1, LED5.VDD, R7.1
- new net N$18: LED6.LEDVDD, R8.2
- new net N$26: C7.1, LED7.VDD, R9.1
- new net N$29: C17.1, LED13.VDD, R1.1
- new net N$35: LED13.LEDVDD, R1.2
- new net N$39: C18.1, LED14.VDD, R2.1
- new net N$40: LED7.LEDVDD, R9.2
- new net N$41: C8.1, LED8.VDD, R10.1
- new net N$46: LED14.LEDVDD, R2.2
- new net N$47: C9.1, LED9.VDD, R11.1
- new net N$48: LED9.LEDVDD, R11.2
- new net N$49: C10.1, LED10.VDD, R12.1
- new net N$50: LED10.LEDVDD, R12.2
- new net N$56: C15.2, U$2.+
- new net N$9: C2.1, LED2.VDD, R4.1
- net GND: now also C17.2, C18.2, LED13.VSS, LED14.VSS; no longer C11.2, C12.2, CN2.GND, CN2.GNDBREAK, LED11.VSS, LED12.VSS
- net N$10: now also LED2.LEDVDD, R4.2; no longer C3.1, LED3.LEDVDD, R3.2
- net N$11: now also C3.1, LED3.VDD, R5.1; no longer C4.1, LED4.LEDVDD, R4.2
- net N$13: now also C4.1, LED4.VDD, R6.1; no longer C5.1, LED5.LEDVDD, R5.2
- net N$14: now also LED4.LEDVDD; no longer C6.1, LED6.LEDVDD
- net N$16: now also LED5.LEDVDD; no longer C7.1, LED7.LEDVDD
- net N$17: now also C6.1, LED6.VDD, R8.1; no longer C8.1, LED8.LEDVDD, R8.2
- net N$19: now also LED13.DI, LED14.DO; no longer C9.1, LED9.LEDVDD, R9.2
- net N$20: now also LED1.DO, LED14.DI; no longer C10.1, LED10.LEDVDD, R10.2
- net N$42: now also LED8.LEDVDD, R10.2; no longer LED10.DI, LED11.DO
- net N$43: now also LED10.DI; no longer LED12.DI
- net N$45: now also U$2.-; no longer C15.2, CN2.PWR1
- net N$7: now also LED1.VDD, R3.1; no longer LED1.LEDVDD, R1.2
- net N$8: now also LED1.LEDVDD, R3.2; no longer C2.1, LED2.LEDVDD, R2.2
- net VCC: no longer LED1.VDD, LED10.VDD, LED11.VDD, LED12.VDD, LED2.VDD, LED3.VDD, LED4.VDD, LED5.VDD, LED6.VDD, LED7.VDD, LED8.VDD, LED9.VDD, R1.1, R10.1, R11.1, R12.1, R2.1, R3.1, R4.1, R5.1, R6.1, R7.1, R8.1, R9.1
Routing:
- net GND: track 311.7 -> 142.7 mm
- net VCC: track 371.5 -> 232.2 mm
- net N$24 (its old number): track 15.5 -> 0.00 mm
- net N$24: track 15.4 -> 0.00 mm
- net N$22: track 15.1 -> 0.00 mm
- net N$53: track 15.1 -> 0.00 mm
- net N$52: track 14.9 -> 0.00 mm
- net N$25: track 14.9 -> 0.00 mm
- net N$55: track 14.7 -> 0.00 mm
- net N$42: track 13.2 -> 0.00 mm
- net N$51: track 13.2 -> 0.00 mm
- net N$21: track 13.1 -> 0.00 mm
- net N$23: track 13.1 -> 0.00 mm
- net N$45: track 20.9 -> 10.4 mm
- net N$13: track 8.46 -> 0.00 mm
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